Commit message: Add files via upload
finished

File: body.urdf (robot description, URDF)
Before this commit: robot robot, 3 links, 2 joints
Links:
- added link BackLeg2, mass 1; collision box size=0.2 0.2 1.0; visual box size=0.2 0.2 1.0
- added link FrontLeg2, mass 1; collision box size=0.2 0.2 1.0; visual box size=0.2 0.2 1.0
- added link LeftLeg, mass 1; collision box size=1.0 0.2 0.2; visual box size=1.0 0.2 0.2
- added link LeftLeg2, mass 1; collision box size=0.2 0.2 1.0; visual box size=0.2 0.2 1.0
- added link RightLeg, mass 1; collision box size=1.0 0.2 0.2; visual box size=1.0 0.2 0.2
- added link RightLeg2, mass 1; collision box size=0.2 0.2 1.0; visual box size=0.2 0.2 1.0
- link Backleg: geometry collision box size=0.2 1 0.2; visual box size=0.2 1 0.2
- link Frontleg: geometry collision box size=0.2 1 0.2; visual box size=0.2 1 0.2
Joints:
- added joint BackLeg_BackLeg2: type revolute, parent Backleg, child BackLeg2, origin xyz=0.0 -1.0 0.0 rpy=0 0 0, axis 1 0 0, limit lower=-3.14159 upper=3.14159 effort=0.0 velocity=0.0
- added joint FrontLeg_FrontLeg2: type revolute, parent Frontleg, child FrontLeg2, origin xyz=0.0 1 0.0 rpy=0 0 0, axis 1 0 0, limit lower=-3.14159 upper=3.14159 effort=0.0 velocity=0.0
- added joint LeftLeg_LeftLeg2: type revolute, parent LeftLeg, child LeftLeg2, origin xyz=1.0 0.0 0.0 rpy=0 0 0, axis 0 1 0, limit lower=-3.14159 upper=3.14159 effort=0.0 velocity=0.0
- added joint RightLeg_RightLeg2: type revolute, parent RightLeg, child RightLeg2, origin xyz=-1.0 0 0.0 rpy=0 0 0, axis 0 1 0, limit lower=-3.14159 upper=3.14159 effort=0.0 velocity=0.0
- added joint Torso_LeftLeg: type revolute, parent Torso, child LeftLeg, origin xyz=0.5 0.0 1.0 rpy=0 0 0, axis 0 1 0, limit lower=-3.14159 upper=3.14159 effort=0.0 velocity=0.0
- added joint Torso_RightLeg: type revolute, parent Torso, child RightLeg, origin xyz=-0.5 0.0 1.0 rpy=0 0 0, axis 0 1 0, limit lower=-3.14159 upper=3.14159 effort=0.0 velocity=0.0
- joint Torso_Backleg: axis 0 1 0 -> 1 0 0; origin xyz=0.5 0 1 rpy=0 0 0 -> xyz=0 -0.5 1 rpy=0 0 0
- joint Torso_Frontleg: axis 0 1 0 -> 1 0 0; origin xyz=-0.5 0 1 rpy=0 0 0 -> xyz=0 0.5 1 rpy=0 0 0
